File: PCB Design/PCB Design.kicad_pcb (KiCad board)
At the start: 2 copper layers, 32.5 x 32.5 mm, 7 parts, among them SW1 SW_Push

Commit message: Routing done
Parts:
- moved R2 7.37 mm to (138.9, 91.4), turned to 180 degrees
Routing:
- net Net-(BT1--): track 0.00 -> 46.3 mm
- net Net-(BT1-+): track 0.00 -> 37.7 mm
- net Net-(D1-K): track 0.00 -> 20.6 mm
- net Net-(D2-A): track 0.00 -> 10.9 mm
- net Net-(D1-A): track 0.00 -> 6.43 mm
Changed lines of the file:
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@@
   )
   (footprint "Resistor_THT:R_Axial_DIN0204_L3.6mm_D1.6mm_P7.62mm_Horizontal" (layer "F.Cu")
-    (at 131.572 91.44)
+    (at 138.938 91.44 180)
     (descr "Resistor, Axial_DIN0204 series, Axial, Horizontal, pin pitch=7.62mm, 0.167W, length*diameter=3.6*1.6mm^2, http://cdn-reichelt.de/documents/datenblatt/B400/1_4W%23YAG.pdf")
     (tags "Resistor Axial_DIN0204 series Axial Horizontal pin pitch 7.62mm 0.167W length 3.6mm diameter 1.6mm")
@@
     (property "ki_keywords" "R res resistor")
     (attr through_hole)
-    (fp_text reference "R2" (at 3.81 -1.92) (layer "F.SilkS")
+    (fp_text reference "R2" (at 3.81 2.032) (layer "F.SilkS")
         (effects (font (size 1 1) (thickness 0.15)))
     )
@@
     (fp_line (start 7.62 0) (end 5.61 0)
       (stroke (width 0.1) (type solid)) (layer "F.Fab"))
-    (pad "1" thru_hole circle (at 0 0) (size 1.4 1.4) (drill 0.7) (layers "*.Cu" "*.Mask")
+    (pad "1" thru_hole circle (at 0 0 180) (size 1.4 1.4) (drill 0.7) (layers "*.Cu" "*.Mask")
       (net 5 "Net-(D2-A)") (pintype "passive"))
-    (pad "2" thru_hole oval (at 7.62 0) (size 1.4 1.4) (drill 0.7) (layers "*.Cu" "*.Mask")
+    (pad "2" thru_hole oval (at 7.62 0 180) (size 1.4 1.4) (drill 0.7) (layers "*.Cu" "*.Mask")
       (net 1 "Net-(BT1-+)") (pintype "passive"))
     (model "${KICAD6_3DMODEL_DIR}/Resistor_THT.3dshapes/R_Axial_DIN0204_L3.6mm_D1.6mm_P7.62mm_Horizontal.wrl"
@@
   (gr_circle (center 134.112 86.36) (end 150.368 86.36)
     (stroke (width 0.1) (type default)) (fill none) (layer "Edge.Cuts"))
+  (segment (start 137.16 78.99) (end 139.192 81.022) (width 0.25) (layer "F.Cu") (net 1))
+  (segment (start 137.16 82.296) (end 135.128 84.328) (width 0.25) (layer "F.Cu") (net 1))
+  (segment (start 129.032 84.328) (end 127 82.296) (width 0.25) (layer "F.Cu") (net 1))
+  (segment (start 127 80.11) (end 128.12 78.99) (width 0.25) (layer "F.Cu") (net 1))
+  (segment (start 135.382 87.376) (end 139.192 87.376) (width 0.25) (layer "F.Cu") (net 1))
+  (segment (start 127 82.296) (end 127 80.11) (width 0.25) (layer "F.Cu") (net 1))
+  (segment (start 131.318 91.44) (end 135.382 87.376) (width 0.25) (layer "F.Cu") (net 1))
+  (segment (start 139.192 81.022) (end 139.192 87.376) (width 0.25) (layer "F.Cu") (net 1))
+  (segment (start 135.128 84.328) (end 129.032 84.328) (width 0.25) (layer "F.Cu") (net 1))
+  (segment (start 137.16 78.99) (end 137.16 82.296) (width 0.25) (layer "F.Cu") (net 1))
+  (segment (start 132.08 77.216) (end 135.128 74.168) (width 0.25) (layer "F.Cu") (net 2))
+  (segment (start 135.128 74.168) (end 140.208 74.168) (width 0.25) (layer "F.Cu") (net 2))
+  (segment (start 132.08 78.99) (end 132.08 77.216) (width 0.25) (layer "F.Cu") (net 2))
+  (segment (start 141.12 78.99) (end 141.12 75.08) (width 0.25) (layer "F.Cu") (net 2))
+  (segment (start 141.12 75.08) (end 140.208 74.168) (width 0.25) (layer "F.Cu") (net 2))
+  (segment (start 132.08 84.328) (end 135.128 87.376) (width 0.25) (layer "B.Cu") (net 2))
+  (segment (start 131.878 99.786) (end 138.378 99.786) (width 0.25) (layer "B.Cu") (net 2))
+  (segment (start 132.08 78.99) (end 132.08 84.328) (width 0.25) (layer "B.Cu") (net 2))
+  (segment (start 135.128 96.536) (end 131.878 99.786) (width 0.25) (layer "B.Cu") (net 2))
+  (segment (start 135.128 87.376) (end 135.128 96.536) (width 0.25) (layer "B.Cu") (net 2))
+  (segment (start 127.798 95.286) (end 123.444 90.932) (width 0.25) (layer "F.Cu") (net 3))
+  (segment (start 138.378 95.286) (end 144.256 89.408) (width 0.25) (layer "F.Cu") (net 3))
+  (segment (start 123.444 89.408) (end 123.444 90.932) (width 0.25) (layer "F.Cu") (net 3))
+  (segment (start 131.878 95.286) (end 127.798 95.286) (width 0.25) (layer "F.Cu") (net 3))
+  (segment (start 144.256 89.408) (end 144.78 89.408) (width 0.25) (layer "F.Cu") (net 3))
+  (segment (start 128.016 87.376) (end 125.984 89.408) (width 0.25) (layer "F.Cu") (net 4))
+  (segment (start 131.572 87.376) (end 128.016 87.376) (width 0.25) (layer "F.Cu") (net 4))
+  (segment (start 147.32 89.408) (end 145.288 87.376) (width 0.25) (layer "F.Cu") (net 5))
+  (segment (start 143.002 87.376) (end 145.288 87.376) (width 0.25) (layer "F.Cu") (net 5))
+  (segment (start 138.938 91.44) (end 143.002 87.376) (width 0.25) (layer "F.Cu") (net 5))
 )
